File: Kinky_NoChop.kicad_pcb (KiCad board)
At the start: 2 copper layers, 80 x 106.7 mm, 313 parts, among them J1 CV_ATT, J10 OUT, J11 OUT, J12 OUT, J13 CV_ATT, J14 VC, J15 IN, J16 OUT, J17 Ctrl, J18 Ctrl, J19 Main, J2 VC, J20 Main, J21 Ctrl, J22 Main, J3 CV_ATT, J4 VC, J5 CV_ATT, J6 VC, J7 IN, J8 IN, J9 IN, Q1 MMBT3906, Q2 MMBT3906, Q3 MMBT3906, Q4 MMBT3906, U1 TL072, U10 TL074, U11 TL074, U12 TL072, U13 TL074, U14 TL074, U2 LM13700, U3 TL074, U4 TL074, U5 TL072, U6 TL074, U7 TL074, U8 TL072, U9 LM13700

Commit message: Worked on the second wavefolder
Routing:
- net Net-(D33-Pad2): track 10.4 -> 24.7 mm, vias 2 -> 3
- net Net-(R68-Pad1): track 12.6 -> 26.4 mm, vias 0 -> 2
- net Net-(D45-Pad2): track 13.9 -> 25.9 mm, vias 0 -> 2
- net Net-(D45-Pad1): track 19.9 -> 29.8 mm, vias 2 -> 4
- net Net-(D39-Pad2): track 2.88 -> 12.4 mm, vias 0 -> 2
- net Net-(D25-Pad2): track 0.00 -> 8.06 mm
- net GND: track 11.0 -> 13.6 mm, vias 14 -> 18
